Commit message: v2.1.0 配置了moveit,能正常跑通moveit的demo

File: my_arm_moveit_config/config/ur3.ros2_control.xacro (robot description, xacro)
@@ -13,5 +13,4 @@
                   <param name="initial_value">${initial_positions['joint1']}</param>
                 </state_interface>
-                <state_interface name="velocity"/>
             </joint>
             <joint name="joint2">
@@ -20,5 +19,4 @@
                   <param name="initial_value">${initial_positions['joint2']}</param>
                 </state_interface>
-                <state_interface name="velocity"/>
             </joint>
             <joint name="joint3">
@@ -27,5 +25,10 @@
                   <param name="initial_value">${initial_positions['joint3']}</param>
                 </state_interface>
-                <state_interface name="velocity"/>
+            </joint>
+            <joint name="joint_tool_gripper">
+                <command_interface name="position"/>
+                <state_interface name="position">
+                  <param name="initial_value">${initial_positions['joint_tool_gripper']}</param>
+                </state_interface>
             </joint>
         </ros2_control>

File: my_robot_description/urdf/ur3.urdf.xacro (robot description, xacro)
@@ -108,4 +108,5 @@
         </collision>
     </link>
+    <link name="tool_link"/>
     <link
         name="gripper">
@@ -171,10 +172,15 @@
         <limit lower="-3.14" upper="3.14" effort="100" velocity="1" />
     </joint>
-    <joint name="joint_gripper" type="revolute">
+    <joint name="joint3_tool" type="fixed">
+        <parent link="link3" />
+        <child link="tool_link" />
+        <origin xyz="0.0 0.0 0.0" rpy="0.0 0.0 0.0"/>
+    </joint>
+    <joint name="joint_tool_gripper" type="revolute">
         <origin xyz="-0.275 0.0 0.055" rpy="-1.5708 0.0 3.1416" />
-        <parent link="link3"/>
+        <parent link="tool_link" />
         <child link="gripper" />
-        <axis xyz="0 0 1"/>
-        <limit lower="0.0" upper="0.0" effort="0.0" velocity="0.0"/>
+        <axis xyz="0 1 0" />
+       <limit lower="-3.14" upper="3.14" effort="100" velocity="1" />
     </joint>
 </robot>
