Commit message: 3.0.0 创建了hardware包并通过了编译

File: my_robot_description/urdf/ur3.ros2_control.xacro (robot description, xacro)
@@ -1,33 +1,41 @@
 <?xml version="1.0"?>
 <robot xmlns:xacro="http://www.ros.org/wiki/xacro">
-        <ros2_control name="Arm" type="system">
-            <hardware>
-                <!-- By default, set up controllers for simulation. This won't work on real hardware -->
-                <plugin>mock_components/GenericSystem</plugin>
-            </hardware>
-            <joint name="joint1">
-                <command_interface name="position"/>
-                <state_interface name="position">
-                  <param name="initial_value">0.0</param>
-                </state_interface>
-            </joint>
-            <joint name="joint2">
-                <command_interface name="position"/>
-                <state_interface name="position">
-                  <param name="initial_value">0.0</param>
-                </state_interface>
-            </joint>
-            <joint name="joint3">
-                <command_interface name="position"/>
-                <state_interface name="position">
-                  <param name="initial_value">0.0</param>
-                </state_interface>
-            </joint>
-            <joint name="joint_tool_gripper">
-                <command_interface name="position"/>
-                <state_interface name="position">
-                  <param name="initial_value">0.0</param>
-                </state_interface>
-            </joint>
-        </ros2_control>
+  <ros2_control name="Arm" type="system">
+    <hardware>
+      <!-- By default, set up controllers for simulation. This won't work on real hardware -->
+      <!-- <plugin>mock_components/GenericSystem</plugin> -->
+      <plugin>arm_hardware_interface/ArmHardwareInterface</plugin>
+    </hardware>
+    <joint name="joint1">
+      <command_interface name="position" />
+      <state_interface name="position">
+        <param name="initial_value">0.0</param>
+      </state_interface>
+    </joint>
+    <joint name="joint2">
+      <command_interface name="position" />
+      <state_interface name="position">
+        <param name="initial_value">0.0</param>
+      </state_interface>
+    </joint>
+    <joint name="joint3">
+      <command_interface name="position" />
+      <state_interface name="position">
+        <param name="initial_value">0.0</param>
+      </state_interface>
+    </joint>
+  </ros2_control>
+  <ros2_control name ="gripper" type="system">
+    <hardware>
+      <!-- By default, set up controllers for simulation. This won't work on real hardware -->
+      <!-- <plugin>mock_components/GenericSystem</plugin> -->
+       <plugin>arm_hardware_interface/ArmHardwareInterface</plugin>
+    </hardware>
+    <joint name="joint_tool_gripper">
+      <command_interface name="position" />
+      <state_interface name="position">
+        <param name="initial_value">0.0</param>
+      </state_interface>
+    </joint>
+  </ros2_control>
 </robot>
